File: Apogee-BK_01_Power/Apogee-BK_01_Power.kicad_sch (KiCad schematic)
At the start: 12 parts, among them J1 Power In (+12VDC), J2 Power Out, U1 PSU5, U2 R-78CK5.0-0.5

Commit message: Added fuse to 12V input rail
Parts:
- added F1: Fuse, Fuse:Fuseholder_Clip-5x20mm_Littelfuse_111_Inline_P20.00x5.00mm_D1.05mm_Horizontal, symbol Device:Fuse
Connections:
- net +12V: now also F1.2; no longer J1.1
- new net +12V_{IN}: F1.1, J1.1
Other:
- note added: "Pin 7 is a fault signal from the motherboard indicating the +5V rail is over/undervoltage. It shuts down the regulators on the orignal power supply ... I think."
- company: (none) -> Brett Hallen
- title: (none) -> Апогей Power Supply
Changed lines of the file:
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@@
 	(generator_version "9.0")
 	(paper "A4")
+	(title_block
+		(title "Апогей Power Supply")
+		(date "14/MAR/2026")
+		(rev "A")
+		(company "Brett Hallen")
+	)
+	(text "Pin 7 is a fault signal from the motherboard indicating the +5V rail is over/undervoltage.\nIt shuts down the regulators on the orignal power supply ... I think."
+		(exclude_from_sim no)
+		(at 161.036 88.138 0)
+		(effects
+			(font
+				(size 1.27 1.27)
+			)
+			(justify left)
+		)
+	)
 	(junction
 		(at 107.95 87.63)
@@
 	(wire
 		(pts
+			(xy 76.2 71.12) (xy 86.36 71.12)
+		)
+		(stroke
+			(width 0)
+			(type default)
+		)
+	)
+	(wire
+		(pts
 			(xy 138.43 60.96) (xy 138.43 58.42)
 		)
@@
 	(wire
 		(pts
-			(xy 76.2 71.12) (xy 97.79 71.12)
-		)
-		(stroke
-			(width 0)
-			(type default)
-		)
-	)
-	(wire
-		(pts
 			(xy 107.95 76.2) (xy 118.11 76.2)
 		)
@@
 		(pts
 			(xy 97.79 71.12) (xy 166.37 71.12)
+		)
+		(stroke
+			(width 0)
+			(type default)
+		)
+	)
+	(wire
+		(pts
+			(xy 93.98 71.12) (xy 97.79 71.12)
 		)
 		(stroke
@@
 		)
 	)
-	(label "+12V"
-		(at 80.01 71.12 0)
+	(label "+12V_{IN}"
+		(at 77.47 71.12 0)
 		(effects
 			(font
@@
 					(unit 1)
 				)
+			)
+		)
+	)
+	(symbol
+		(lib_id "Device:Fuse")
+		(at 90.17 71.12 90)
+		(unit 1)
+		(exclude_from_sim no)
+		(in_bom yes)
+		(on_board yes)
+		(dnp no)
+		(fields_autoplaced yes)
+		(property "Reference" "F1"
+			(at 90.17 64.77 90)
+			(effects
+				(font
+					(size 1.27 1.27)
+				)
+			)
+		)
+		(property "Value" "Fuse"
+			(at 90.17 67.31 90)
+			(effects
+				(font
+					(size 1.27 1.27)
+				)
+			)
+		)
+		(property "Footprint" "Fuse:Fuseholder_Clip-5x20mm_Littelfuse_111_Inline_P20.00x5.00mm_D1.05mm_Horizontal"
+			(at 90.17 72.898 90)
+			(effects
+				(font
+					(size 1.27 1.27)
+				)
+				(hide yes)
+			)
+		)
+		(property "Datasheet" "~"
+			(at 90.17 71.12 0)
+			(effects
+				(font
+					(size 1.27 1.27)
+				)
+				(hide yes)
+			)
+		)
+		(property "Description" "Fuse"
+			(at 90.17 71.12 0)
+			(effects
+				(font
+					(size 1.27 1.27)
+				)
+				(hide yes)
+			)
+		)
+		(pin "1"
+		)
+		(pin "2"
+		)
+		(instances
+			(project ""
+				(path "/bff640d3-88e6-45d7-956e-e9c03bf1b325"
+					(reference "F1")
+					(unit 1)
+				)
